File: anac_2040.kicad_pcb (KiCad board)
At the start: 2 copper layers, 53.2 x 68.2 mm, 62 parts, among them J1 Conn_01x02, J10 Debug, J5 Conn_01x09, J6 Barrel_Jack_MountingPin, J7 USB_C_Receptacle_USB2.0, Q1 PJA3432AU, Q2 PJA3432AU, SW1 SW_Push, SW2 SW_Push, U1 RP2040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

Commit message: fixed things
Parts:
- moved C13 0.10 mm to (152.9, 112.0)
- moved C14 0.10 mm to (154.9, 112.0)
- moved C16 0.07 mm to (155.2, 66.8)
Routing:
- net +3.3V: track 160.2 -> 160.9 mm

Commit message: few fixes
Parts:
- added Fuse bypass: Jumper, Jumper:SolderJumper-2_P1.3mm_Open_RoundedPad1.0x1.5mm, F.Cu at (160.1, 58.2)
- moved D1 0.90 mm to (157.2, 58.9)
- moved F1 0.45 mm to (159.0, 62.2)
Routing:
- net VBUS: track 14.8 -> 18.0 mm
- net +3.3V: track 160.9 -> 159.4 mm, vias 4 -> 3
- net VBUSPIN: track 45.6 -> 47.0 mm
- net VSYS: track 77.6 -> 76.3 mm
- net GND1: track 119.5 -> 118.5 mm, vias 4 -> 2
- net DP: track 24.7 -> 25.6 mm
- net D-: track 40.6 -> 40.0 mm
- net GPIO29: track 56.9 -> 56.4 mm
- net GND: vias 20 -> 16
Other:
- board text added: "D+"
- board text added: "D-"
- board text added: "Fuse bypass Max 1A"

Commit message: i forget
Parts:
- moved R1 1.50 mm to (147.3, 89.6)
- moved C18 0.45 mm to (143.2, 73.4)
- moved C19 0.45 mm to (148.2, 73.4)
- moved J1 0.45 mm to (145.7, 62.5)
- moved J6 0.25 mm to (136.2, 66.2)
Routing:
- net +3.3V: track 159.4 -> 158.1 mm
- net GPIO24: track 66.8 -> 65.6 mm
- net Net-(C2-Pad2): track 11.1 -> 10.00 mm
- net Net-(R1-Pad1): track 12.0 -> 11.0 mm
- net VBUS: track 18.0 -> 18.9 mm
- net VSYS: track 76.3 -> 75.7 mm
- net GND1: track 118.5 -> 118.0 mm, vias 2 -> 1
- net GND: track 4.29 -> 3.79 mm
Other:
- board text added: "1,1V"
- board text added: "3,3V"
- board text added: "3,8-33V"
- board text added: "Fuse bypass Max 2A"
- board text removed: "1,1v"
- board text removed: "3,3v"
- board text removed: "Fuse bypass Max 1A"

Commit message: small design change
Routing:
- net +3.3V: track 158.1 -> 153.2 mm
- net VSYS: track 75.7 -> 74.4 mm
- net GPIO13: track 39.4 -> 38.5 mm
- net GPIO15: track 48.0 -> 48.6 mm
- net GND: vias 16 -> 18
Other:
- board text added: "3,8-32V"
- board text removed: "3,8-33V"

Commit message: mix
Parts:
- moved C7 4.48 mm to (160.3, 116.1), turned to 180 degrees
- moved C15 3.22 mm to (158.1, 118.6), turned to -90 degrees
- moved C13 2.67 mm to (153.7, 109.4), turned to 180 degrees
- moved C8 1.89 mm to (148.6, 97.0)
- moved C14 1.61 mm to (153.7, 110.9), turned to 180 degrees
- moved C5 1.51 mm to (148.6, 98.5)
- moved R12 1.16 mm to (159.7, 118.6)
- moved R1 0.57 mm to (147.3, 90.1)
Routing:
- net +3.3V: track 153.2 -> 146.8 mm
- net GPIO25: track 98.7 -> 94.3 mm
- net RST: track 80.4 -> 83.9 mm
- net +1V1: track 57.2 -> 55.0 mm
- net Net-(D5-Pad1): track 6.30 -> 4.64 mm
- net QSPI_SS: track 45.3 -> 46.6 mm
- net GND1: track 117.9 -> 117.0 mm
- net GPIO24: track 65.6 -> 64.6 mm
- net Net-(D4-Pad2): track 5.79 -> 4.84 mm
- net SWD: track 35.4 -> 36.2 mm
- net Net-(C2-Pad2): track 10.00 -> 10.6 mm
- net Net-(R1-Pad1): track 11.0 -> 10.4 mm

Commit message: stuff
Parts:
- removed J1: Conn_01x02, DIY:WAGO SMD terminal, 2P 4mm
- added REF**: Symbol_Barrel_Polarity, Symbol:Symbol_Barrel_Polarity, F.Cu at (142.7, 61.1)
- C1, C10, C11, C12, C13, C14, C15, C16, C2, C3, C4, C5, C6, C7, C8, C9: footprint Capacitor_SMD:C_0603_1608Metric -> Capacitor_SMD:C_0402_1005Metric
- D2, D3, D4: footprint LED_SMD:LED_0603_1608Metric -> LED_SMD:LED_0402_1005Metric
- JP1: renamed from Fuse bypass
- R1, R10, R11, R12, R13, R14, R15, R16, R17, R2, R3, R4, R5, R6, R7, R8, R9, RV1, RV2: footprint Resistor_SMD:R_0603_1608Metric -> Resistor_SMD:R_0402_1005Metric
- moved C19 4.55 mm to (147.2, 68.9), turned to 180 degrees
- moved C18 4.10 mm to (147.2, 73.9), turned to 180 degrees
Connections:
- net 3,3V_EN renamed Net-(U4-EN)
Routing:
- net VSYS: track 74.4 -> 49.9 mm
- net GND1: track 117.0 -> 96.9 mm
- net +3.3V: track 146.8 -> 151.6 mm
- net GPIO16: track 31.6 -> 28.6 mm
- net GPIO15: track 48.6 -> 45.9 mm
- net GPIO17: track 23.9 -> 22.4 mm
- net GPIO18: track 21.0 -> 20.3 mm
Other:
- board text added: "Anna2040 v1,3"
- board text removed: "Anna2040 v1,2"
