File: anac_2040.kicad_sch (KiCad schematic)
At the start: 62 parts, among them J1 Conn_01x02, J10 Debug, J5 Conn_01x09, J6 Barrel_Jack_MountingPin, J7 USB_C_Receptacle_USB2.0, Q1 PJA3432AU, Q2 PJA3432AU, SW1 SW_Push, SW2 SW_Push, U1 RP2040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

Commit message: small update
Parts:
- removed D1: D_Schottky, Diode_SMD:D_SOD-323, symbol Device:D_Schottky_Small
- added D1: D_Small, Diode_SMD:D_SOD-323, symbol Device:D_Small
- C1, C10, C11, C12, C13, C14, C15, C16, C2, C3, C4, C5, C6, C7, C8, C9: footprint Capacitor_SMD:C_0805_2012Metric -> Capacitor_SMD:C_0603_1608Metric
- D2, D3, D4: footprint LED_SMD:LED_0805_2012Metric -> LED_SMD:LED_0603_1608Metric
- J1: footprint DIY:WAGO terminal, 2P 3mm -> DIY:WAGO SMD terminal, 2P 4mm
- R1, R10, R11, R12, R13, R14, R15, R16, R17, R2, R3, R4, R5, R6, R7, R8, R9, RV1, RV2: footprint Resistor_SMD:R_0805_2012Metric -> Resistor_SMD:R_0603_1608Metric
Connections:
- net GND1: now also J1.1 (Pin_1); no longer J1.2 (Pin_2)
- net VBUSPIN: now also D1.2 (A)
- net VSYS: now also J1.2 (Pin_2), D1.1 (K); no longer J1.1 (Pin_1)

Commit message: few fixes
Parts:
- added JP1: Jumper, Jumper:SolderJumper-2_P1.3mm_Open_RoundedPad1.0x1.5mm, symbol Jumper:SolderJumper_2_Open
Connections:
- net VBUS: now also JP1.1 (A)
- net VBUSPIN: now also JP1.2 (B)
Other:
- moved on the sheet: F1
Changed lines of the file:
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@@
   (junction (at 97.79 24.13) (diameter 0) (color 0 0 0 0)
   )
+  (junction (at 153.67 36.83) (diameter 0) (color 0 0 0 0)
+  )
   (junction (at 213.36 95.25) (diameter 0) (color 0 0 0 0)
   )
@@
   (junction (at 248.92 67.31) (diameter 0) (color 0 0 0 0)
   )
+  (junction (at 143.51 36.83) (diameter 0) (color 0 0 0 0)
+  )
   (junction (at 161.29 163.83) (diameter 0) (color 0 0 0 0)
   )
@@
     (stroke (width 0) (type default) (color 0 0 0 0))
   )
+  (wire (pts (xy 152.4 39.37) (xy 153.67 39.37))
+    (stroke (width 0) (type default) (color 0 0 0 0))
+  )
   (wire (pts (xy 125.73 127) (xy 129.54 127))
     (stroke (width 0) (type default) (color 0 0 0 0))
@@
     (stroke (width 0) (type default) (color 0 0 0 0))
   )
+  (wire (pts (xy 153.67 36.83) (xy 153.67 39.37))
+    (stroke (width 0) (type default) (color 0 0 0 0))
+  )
   (wire (pts (xy 116.84 24.13) (xy 116.84 25.4))
     (stroke (width 0) (type default) (color 0 0 0 0))
@@
     (stroke (width 0) (type default) (color 0 0 0 0))
   )
+  (wire (pts (xy 144.78 39.37) (xy 143.51 39.37))
+    (stroke (width 0) (type default) (color 0 0 0 0))
+  )
   (wire (pts (xy 276.86 144.78) (xy 276.86 142.24))
     (stroke (width 0) (type default) (color 0 0 0 0))
@@
     (stroke (width 0) (type default) (color 0 0 0 0))
   )
-  (wire (pts (xy 143.51 36.83) (xy 146.05 36.83))
+  (wire (pts (xy 142.24 36.83) (xy 143.51 36.83))
     (stroke (width 0) (type default) (color 0 0 0 0))
   )
@@
     (stroke (width 0) (type default) (color 0 0 0 0))
   )
-  (wire (pts (xy 153.67 36.83) (xy 154.94 36.83))
+  (wire (pts (xy 152.4 36.83) (xy 153.67 36.83))
     (stroke (width 0) (type default) (color 0 0 0 0))
   )
@@
     (stroke (width 0) (type default) (color 0 0 0 0))
   )
+  (wire (pts (xy 153.67 36.83) (xy 154.94 36.83))
+    (stroke (width 0) (type default) (color 0 0 0 0))
+  )
+  (wire (pts (xy 143.51 36.83) (xy 144.78 36.83))
+    (stroke (width 0) (type default) (color 0 0 0 0))
+  )
   (wire (pts (xy 270.51 64.77) (xy 270.51 66.04))
     (stroke (width 0) (type default) (color 0 0 0 0))
@@
     (stroke (width 0) (type default) (color 0 0 0 0))
   )
+  (wire (pts (xy 143.51 36.83) (xy 143.51 39.37))
+    (stroke (width 0) (type default) (color 0 0 0 0))
+  )
   (wire (pts (xy 101.6 31.75) (xy 101.6 30.48))
     (stroke (width 0) (type default) (color 0 0 0 0))
@@
     )
   )
-  (global_label "VBUS" (shape input) (at 143.51 36.83 180) (fields_autoplaced)
+  (global_label "VBUS" (shape input) (at 142.24 36.83 180) (fields_autoplaced)
     (effects (font (size 1.27 1.27)) (justify right))
-    (property "Intersheet References" "${INTERSHEET_REFS}" (id 0) (at 136.1983 36.7506 0)
+    (property "Intersheet References" "${INTERSHEET_REFS}" (id 0) (at 134.9283 36.7506 0)
       (effects (font (size 1.27 1.27)) (justify right) hide)
     )
@@
     (pin "1")
   )
+  (symbol (lib_id "Jumper:SolderJumper_2_Open") (at 148.59 39.37 0) (unit 1)
+    (in_bom yes) (on_board yes)
+    (property "Reference" "JP1" (id 0) (at 140.97 40.64 0))
+    (property "Value" "Jumper" (id 1) (at 140.97 43.18 0))
+    (property "Footprint" "Jumper:SolderJumper-2_P1.3mm_Open_RoundedPad1.0x1.5mm" (id 2) (at 148.59 39.37 0)
+      (effects (font (size 1.27 1.27)) hide)
+    )
+    (property "Datasheet" "~" (id 3) (at 148.59 39.37 0)
+      (effects (font (size 1.27 1.27)) hide)
+    )
+    (pin "1")
+    (pin "2")
+  )
   (symbol (lib_id "Connector:Conn_01x02_Female") (at 41.91 26.67 0) (mirror x) (unit 1)
     (in_bom yes) (on_board yes)
@@
     (pin "2")
   )
-  (symbol (lib_id "Device:Fuse") (at 149.86 36.83 270) (unit 1)
+  (symbol (lib_id "Device:Fuse") (at 148.59 36.83 270) (unit 1)
     (in_bom yes) (on_board yes)
-    (property "Reference" "F1" (id 0) (at 151.13 31.75 90)
+    (property "Reference" "F1" (id 0) (at 149.86 31.75 90)
       (effects (font (size 1.27 1.27)) (justify right))
     )
-    (property "Value" "500mA" (id 1) (at 152.4 34.2901 90)
+    (property "Value" "500mA" (id 1) (at 151.13 34.2901 90)
       (effects (font (size 1.27 1.27)) (justify right))
     )
-    (property "Footprint" "Fuse:Fuse_1206_3216Metric" (id 2) (at 149.86 35.052 90)
+    (property "Footprint" "Fuse:Fuse_1206_3216Metric" (id 2) (at 148.59 35.052 90)
       (effects (font (size 1.27 1.27)) hide)
     )
-    (property "Datasheet" "~" (id 3) (at 149.86 36.83 0)
+    (property "Datasheet" "~" (id 3) (at 148.59 36.83 0)
       (effects (font (size 1.27 1.27)) hide)
     )
@@
       (reference "J10") (unit 1) (value "Debug") (footprint "Connector_PinSocket_2.54mm:PinSocket_1x03_P2.54mm_Vertical")
     )
+    (path "/4dd0a9cf-1b92-4e2c-9867-fbfa3bd8e862"
+      (reference "JP1") (unit 1) (value "Jumper") (footprint "Jumper:SolderJumper-2_P1.3mm_Open_RoundedPad1.0x1.5mm")
+    )
     (path "/55aa6bdf-66e4-45b7-91d3-47fa6b2d57b6"

Commit message: i forget
Connections:
- net 3,3V_EN: no longer names the net of R9.2, U4.2 (EN)
Changed lines of the file:
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@@
   (junction (at 224.79 143.51) (diameter 0) (color 0 0 0 0)
   )
-  (junction (at 175.26 46.99) (diameter 0) (color 0 0 0 0)
-  )
   (junction (at 33.02 20.32) (diameter 0) (color 0 0 0 0)
   )
@@
   )
   (wire (pts (xy 162.56 36.83) (xy 162.56 39.37))
-    (stroke (width 0) (type default) (color 0 0 0 0))
-  )
-  (wire (pts (xy 173.99 46.99) (xy 175.26 46.99))
     (stroke (width 0) (type default) (color 0 0 0 0))
   )
@@
     )
   )
-  (global_label "3,3V_EN" (shape input) (at 173.99 46.99 180) (fields_autoplaced)
-    (effects (font (size 1.27 1.27)) (justify right))
-    (property "Intersheet References" "${INTERSHEET_REFS}" (id 0) (at 164.0174 46.9106 0)
-      (effects (font (size 1.27 1.27)) (justify right) hide)
-    )
-  )

Commit message: stuff
Parts:
- removed J1: Conn_01x02, DIY:WAGO SMD terminal, 2P 4mm, symbol Connector:Conn_01x02_Female
- C1, C10, C11, C12, C13, C14, C15, C16, C2, C3, C4, C5, C6, C7, C8, C9: footprint Capacitor_SMD:C_0603_1608Metric -> Capacitor_SMD:C_0402_1005Metric
- D2, D3, D4: footprint LED_SMD:LED_0603_1608Metric -> LED_SMD:LED_0402_1005Metric
- R1, R10, R11, R12, R13, R14, R15, R16, R17, R2, R3, R4, R5, R6, R7, R8, R9, RV1, RV2: footprint Resistor_SMD:R_0603_1608Metric -> Resistor_SMD:R_0402_1005Metric
Other:
- note added: "Current leakage prevention"
- note removed: "Power selector maybe ¯\_(ツ)_/¯"
